File: board/board-eagle/snowflake.brd (EAGLE design)
At the start: 67.5 x 65.8 mm, 9 parts, among them U1 Tiny85-20-SMT

Commit message: new board and zip
Parts:
- U1: value Tiny85-20-SMT -> (none)
Connections:
- net MISO: now also D1.2, D2.2, D3.2, D4.2, D5.2
- net VCC: no longer D1.2, D2.2, D3.2, D4.2, D5.2
Routing:
- net MISO: track 15.1 -> 157.3 mm, vias 1 -> 0
- net VCC: track 180.0 -> 65.5 mm, vias 0 -> 2
- net N$1: track 64.3 -> 0.25 mm, vias 3 -> 1
- net GND: track 91.2 -> 61.0 mm
- net SCK: track 21.3 -> 12.9 mm, vias 1 -> 0
- net MOSI: track 32.1 -> 24.9 mm
- net RESET: track 29.0 -> 25.3 mm
- net N$2: track 49.1 -> 46.9 mm
- net N$4: track 45.2 -> 46.8 mm
- net N$5: track 48.3 -> 49.6 mm
- net N$13: track 0.00 -> 0.61 mm, vias 0 -> 1
- net N$14: track 0.00 -> 0.39 mm, vias 0 -> 1
Other:
- board text added: "XMAS 2016"
